File: kicad/thesis/_autosave-thesis.kicad_sch (KiCad schematic)
At the start: 14 parts, among them Q1 IRLZB8721, SW1 SW_DIP_x01, U1 INA219AxD

Commit message: Added PCB Design
Made folder for the electromagnet placeholder pins. (Note: download arduino extension to get the footprint for the BLE 33 Sense)
Parts:
- L1, L2: footprint (none) -> Personalized-footprint:Iron-Input
- L3, L4: footprint (none) -> Personalized-footprint:Iron-Output
Other:
- moved on the sheet: A1, D1, D2, L1, L2, L3, L4, Q1, R1, R2, R3, SW1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
